File: Shiba 2.kicad_pcb (KiCad board)
At the start: 2 copper layers, 85.7 x 54 mm, 59 parts, among them J1 Conn_01x06_Pin, J2 Jack-DC, J3 Conn_01x010_Pin, SW1 SW_SPDT, U1 AP62150Z6, U2 MIC5504-3.3YM5, U3 STM32F072C8Tx

Commit message: Rev 2 maybe?
Parts:
- removed U3: STM32F072C8Tx, Package_QFP:LQFP-48_7x7mm_P0.5mm
- added C14: C2.2uF, Capacitor_SMD:C_1206_3216Metric_Pad1.33x1.80mm_HandSolder, F.Cu at (115.1, 61.3)
- added C16: C1uF, Capacitor_SMD:C_1206_3216Metric_Pad1.33x1.80mm_HandSolder, F.Cu at (117.6, 61.3)
- added C9: C2.2uF, Capacitor_SMD:C_1206_3216Metric_Pad1.33x1.80mm_HandSolder, F.Cu at (111.3, 46.5)
- added J4: Conn_01x02_Pin, Connector_PinHeader_2.54mm:PinHeader_1x02_P2.54mm_Vertical, F.Cu at (104.5, 51.8)
- added J5: Conn_01x03_Pin, Connector_PinSocket_2.54mm:PinSocket_1x03_P2.54mm_Vertical, F.Cu at (80.6, 33.3)
- added J6: Conn_01x03_Pin, Connector_PinSocket_2.54mm:PinSocket_1x03_P2.54mm_Vertical, F.Cu at (77.8, 33.3)
- added J7: Conn_01x03_Pin, Connector_PinSocket_2.54mm:PinSocket_1x03_P2.54mm_Vertical, F.Cu at (75.0, 33.3)
- added J8: Conn_01x03_Pin, Connector_PinSocket_2.54mm:PinSocket_1x03_P2.54mm_Vertical, F.Cu at (72.2, 33.3)
- added U4: STM32H503CBTx, Package_QFP:LQFP-48_7x7mm_P0.5mm, F.Cu at (113.3, 53.1)
- J3: value Conn_01x010_Pin -> GPIO; footprint Connector_PinSocket_2.54mm:PinSocket_1x10_P2.54mm_Vertical -> Connector_PinSocket_2.54mm:PinSocket_1x08_P2.54mm_Vertical
- moved J3 53.6 mm to (82.5, 48.0)
- moved R11 15.7 mm to (116.5, 46.2), turned to 0 degrees
- moved J1 13.3 mm to (120.8, 61.2), turned to 180 degrees
- moved C2 11.7 mm to (107.3, 47.5), turned to 90 degrees
- moved C6 11.3 mm to (74.9, 50.3), turned to 180 degrees
- moved L3 7.96 mm to (77.0, 44.5), turned to -90 degrees
- moved C7 6.76 mm to (70.9, 55.5), turned to 90 degrees
- moved R3 6.47 mm to (69.6, 59.5)
- moved C5 6.06 mm to (77.0, 55.5), turned to -90 degrees
- moved C4 5.82 mm to (73.2, 43.2), turned to 180 degrees
- moved R4 5.59 mm to (109.0, 61.0), turned to 0 degrees
- moved SW1 5.48 mm to (105.0, 63.2)
- moved C12 5.12 mm to (130.6, 60.7), turned to 0 degrees
- moved D8 4.87 mm to (87.0, 51.3)
- moved D7 4.87 mm to (89.5, 51.3)
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Connections:
- net IC21_SCL renamed I2C1_SCL
- J3 pad 1: GPIO_7 -> GPIO_5
- J3 pad 2: GPIO_6 -> GPIO_4
- J3 pad 3: GPIO_5 -> GPIO_3
- J3 pad 4: GPIO_4 -> GPIO_2
- J3 pad 5: GPIO_3 -> GPIO_1
- J3 pad 6: GPIO_2 -> GPIO_0
- J3 pad 7: GPIO_1 -> GND
- J3 pad 8: GPIO_0 -> +3V3
Routing:
- net +3V3: track 238.4 -> 98.9 mm, vias 5 -> 7
- net SERVO_3: track 0.00 -> 65.4 mm, vias 0 -> 1
- net +BATT: track 14.9 -> 79.6 mm, vias 4 -> 3
- net SERVO_2: track 0.00 -> 62.4 mm, vias 0 -> 1
- net SERVO_1: track 0.00 -> 55.2 mm, vias 0 -> 1
- net SERVO_0: track 0.00 -> 50.8 mm, vias 0 -> 1
- net GPIO_7: track 32.3 -> 0.00 mm, vias 2 -> 0
- net GPIO_6: track 29.2 -> 0.00 mm, vias 2 -> 0
- net IMU_INT: track 19.7 -> 0.00 mm, vias 2 -> 0
- net GPIO_4: track 47.2 -> 28.2 mm
- net GND: track 22.5 -> 4.28 mm, vias 5 -> 2
- net GPIO_3: track 44.8 -> 30.3 mm
- net GPIO_2: track 42.4 -> 29.2 mm
- net TIM3_CH2: track 14.6 -> 26.3 mm, vias 0 -> 1
- net TIM1_CH1: track 10.3 -> 20.9 mm, vias 0 -> 1
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- added copper zone on B.Cu, net +3V3
Other:
- board text added: "RX"
- board text added: "SERVOS"
- board text added: "TX"
- board text added: "UART"
- board text removed: "6"
- board text removed: "7"

Commit message: more rev2 revisions
Parts:
- moved Battery1 15.0 mm to (61.0, 51.8), turned to -90 degrees
- moved J2 5.11 mm to (64.8, 42.4), turned to 180 degrees
- moved R1 2.87 mm to (69.1, 50.5), turned to 90 degrees
- moved C1 1.85 mm to (109.7, 43.4)
- moved C4 1.55 mm to (73.5, 44.7)
- moved C6 1.55 mm to (75.1, 51.8)
- moved U1 1.55 mm to (74.5, 47.1)
- moved C3 1.55 mm to (71.4, 48.5)
- moved R2 1.55 mm to (75.2, 49.5)
- moved L3 1.55 mm to (77.2, 46.0)
- moved R3 1.43 mm to (70.4, 60.7)
- moved C5 1.30 mm to (76.5, 56.7)
- moved U2 1.30 mm to (73.4, 56.7)
- moved C7 1.30 mm to (70.4, 56.7)
- moved R10 1.19 mm to (87.0, 56.4)
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Routing:
- net +BATT: track 79.6 -> 65.6 mm
- net +5V: track 99.6 -> 102.1 mm
- net Net-(D1-A): track 7.16 -> 5.13 mm
- net Net-(D8-K): track 3.38 -> 2.01 mm
- net Net-(D7-K): track 3.38 -> 2.01 mm
- net Net-(D6-K): track 3.38 -> 2.01 mm
- net Net-(D5-K): track 3.38 -> 2.01 mm
- net Net-(D4-K): track 3.38 -> 2.01 mm
- net Net-(D3-K): track 3.38 -> 2.01 mm
- net Net-(U1-FB): track 6.75 -> 7.81 mm
- net Net-(U1-SW): track 5.41 -> 6.09 mm
- removed copper zone on B.Cu, net +BATT
