File: Sheba 2.kicad_sch (KiCad schematic)
At the start: 64 parts, among them J1 Conn_01x06_Pin, J2 Jack-DC, J3 GPIO, J4 Conn_01x02_Pin, J5 Conn_01x03_Pin, J6 Conn_01x03_Pin, J7 Conn_01x03_Pin, J8 Conn_01x03_Pin, SW1 SW_SPDT, U1 AP62150Z6, U2 MIC5504-3.3YM5, U4 STM32H503CBTx

Commit message: Preparing to remove USB port and switch to STM32F072CBTx
Parts:
- added C14: C1uF, Capacitor_SMD:C_1206_3216Metric_Pad1.33x1.80mm_HandSolder, symbol Device:C_Small
- renumbered C4 to C1, C6 to C10, C7 to C12, C5 to C13, C12 to C15, C14 to C16, C16 to C17, C1 to C2, C9 to C3, C2 to C4, C10 to C5, C8 to C6, C15 to C7, C3 to C8, C13 to C9, D8 to D1, D7 to D2, D6 to D3, D5 to D4, D4 to D5, D3 to D6, D1 to D7, D2 to D8, EP2 to EP1, EP3 to EP2, EP1 to EP3, J8 to J1, J7 to J2, J6 to J3, J5 to J4, J2 to J5, J3 to J6, J1 to J7, J4 to J8, L3 to L1, R11 to R1, R6 to R10, R5 to R11, R3 to R12, R4 to R13, R1 to R2, R2 to R3, R12 to R4, R13 to R5, R10 to R6, R9 to R7, R7 to R9, U4 to U2, U2 to U3
Connections:
- net +3V3: now also C14.2
- net GND: now also C14.1
- net IMU_INT: now also U2.31 (PA10)
- net M3_OUT2: now reaches MD1.1 (OUT1), Motor Terminal1.6 (Pin_6)
- net M3_OUT1: now reaches MD1.7 (OUT2), Motor Terminal1.5 (Pin_5)
- net M2_OUT2: now reaches MD2.1 (OUT1), Motor Terminal1.4 (Pin_4)
- net M2_OUT1: now reaches MD2.7 (OUT2), Motor Terminal1.3 (Pin_3)
- net M1_OUT2: now reaches MD3.1 (OUT1), Motor Terminal1.2 (Pin_2)
- net M1_OUT1: now reaches MD3.7 (OUT2), Motor Terminal1.1 (Pin_1)
- no-connect marks 6 -> 8
Other:
- note added: "STM32"
- title: Shiba 2 -> Sheba 2
- moved on the sheet: C16, C17, C2, C3, C4, R1, U2, USB_A1
Changed lines of the file:
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@@
 	(paper "A3")
 	(title_block
-		(title "Shiba 2")
+		(title "Sheba 2")
+		(date "2024-04-23")
 		(rev "1")
 		(company "Lorem Ipsum Automation")

Commit message: Rev 2 ordered!
Parts:
- removed C16, C3: C2.2uF, Capacitor_SMD:C_1206_3216Metric_Pad1.33x1.80mm_HandSolder, symbol Device:C_Small
- removed J1: Conn_01x03_Pin, Connector_PinSocket_2.54mm:PinSocket_1x03_P2.54mm_Vertical, symbol Connector:Conn_01x03_Pin
- removed J5: Jack-DC, Connector_BarrelJack:BarrelJack_CUI_PJ-063AH_Horizontal, symbol Connector:Jack-DC
- removed J6: GPIO, Connector_PinSocket_2.54mm:PinSocket_1x08_P2.54mm_Vertical, symbol Connector:Conn_01x08_Pin
- removed U2: STM32H503CBTx, Package_QFP:LQFP-48_7x7mm_P0.5mm, symbol MCU_ST_STM32H5:STM32H503CBTx
- removed USB_A1: USB_A, Connector_USB:USB_A_Receptacle_GCT_USB1046, symbol Connector:USB_A
- added J9: Conn_02x04_Top_Bottom, Connector_PinSocket_2.54mm:PinSocket_2x04_P2.54mm_Vertical, symbol Connector_Generic:Conn_02x04_Top_Bottom
- added P1: USB_C_Plug_USB2.0, Connector_USB:USB_C_Receptacle_GCT_USB4105-xx-A_16P_TopMnt_Horizontal, symbol Connector:USB_C_Plug_USB2.0
- added R14: R10k, Resistor_SMD:R_1206_3216Metric_Pad1.30x1.75mm_HandSolder, symbol Device:R
- added U4: STM32F072CBTx, Package_QFP:LQFP-48_7x7mm_P0.5mm, symbol MCU_ST_STM32F0:STM32F072CBTx
- EP1, EP2, EP3, J2, J3, J4, J8: DigiKey 2.54mm Pin Socket -> (none)
- J7: DigiKey 2.54mm Pin Header -> (none)
- R1: value R10k -> 5.11K; DigiKey RC1206FR-0710KL -> P150BCCT-ND
Connections:
- net +3V3: now also C17.1, C2.2, J9.1 (Pin_1), U4.1 (VBAT), U4.24 (VDD), U4.36 (VDDIO2), U4.48 (VDD), U4.9 (VDDA); no longer C17.2, C2.1
- net +5V: now also P1.A4 (VBUS), P1.A9 (VBUS), P1.B4 (VBUS), P1.B5 (VCONN), P1.B9 (VBUS)
- net BLINKY: now also U4.25 (PB12)
- net BOOT0: now also R14.1, U4.44 (BOOT0); no longer R1.1
- net GND: now also C17.2, C2.1, R1.1, J9.2 (Pin_2), P1.A1 (GND), P1.A12 (GND), P1.B1 (GND), P1.B12 (GND), P1.S1 (SHIELD), R14.2, U4.23 (VSS), U4.35 (VSS), U4.47 (VSS), U4.8 (VSSA); no longer C17.1, C2.2, R1.2
- net IMU_INT: now also U4.28 (PB15)
- net KIWI_DRIVE: now also U4.20 (PB2)
- net M1_FWD: now also U4.10 (PA0)
- net M1_REV: now also U4.11 (PA1)
- net M2_FWD: now also U4.12 (PA2)
- net M2_REV: now also U4.13 (PA3)
- net M3_FWD: now also U4.14 (PA4)
- net M3_REV: now also U4.15 (PA5)
- net NRST: now also J7.3 (Pin_3), U4.7 (NRST); no longer J7.5 (Pin_5)
- net SYS_SWCLK: now also J7.5 (Pin_5), U4.37 (PA14); no longer J7.4 (Pin_4)
- net SYS_SWDIO: now also J7.4 (Pin_4), U4.34 (PA13); no longer J7.3 (Pin_3)
- net TIM1_CH1: now also U4.29 (PA8)
- net TIM1_CH2: now also U4.30 (PA9)
- net TIM2_CH1: now also U4.38 (PA15)
- net TIM2_CH2: now also U4.39 (PB3)
- net TIM3_CH1: now also U4.40 (PB4)
- net TIM3_CH2: now also U4.41 (PB5)
- net USB_D+: now also P1.A6 (D+), U4.33 (PA12)
- net USB_D-: now also P1.A7 (D-), U4.32 (PA11)
- net I2C1_SCL renamed I2C2_SCL
- net I2C2_SCL: now also U4.26 (PB13)
- net I2C1_SDA renamed I2C2_SDA
- net I2C2_SDA: now also U4.27 (PB14)
- net SERVO_0 renamed SERVO0
- net SERVO0: now also U4.17 (PA7)
- net SERVO_1 renamed SERVO1
- net SERVO1: now also U4.16 (PA6)
- net SERVO_2 renamed SERVO2
- net SERVO2: now also U4.31 (PA10)
- net USART1_RX renamed USART3_RX
- net USART3_RX: now also U4.22 (PB11)
- net USART1_TX renamed USART3_TX
- net USART3_TX: now also U4.21 (PB10)
- new net: P1.A5 (CC), R1.2
- new net GPIO0: J9.3 (Pin_3), U4.42 (PB6)
- new net GPIO1: J9.5 (Pin_5), U4.43 (PB7)
- new net GPIO2: J9.7 (Pin_7), U4.46 (PB9)
- new net GPIO3: J9.8 (Pin_8), U4.2 (PC13)
- new net GPIO4: J9.6 (Pin_6), U4.3 (PC14)
- new net GPIO5: J9.4 (Pin_4), U4.4 (PC15)
- no-connect marks 8 -> 11
Other:
- note added: "AP_CS wired to VDD for I2C mode"
- note added: "Debug Port"
- note added: "GPIO"
- note added: "I2C Pull-ups"
- note added: "Servo Ports"
- note added: "UART"
- note added: "USB Type C Port"
- moved on the sheet: Battery1, C1, C13, C8, D1, D2, D3, D4, D5, D6, D7, D8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

Commit message: Post-rev 2 changes
Parts:
- Battery1: value ~ -> XT-60
- EP1, EP2, EP3, J2, J3, J4, J7, J8, J9: now not fitted
- Motor Terminal1: value ~ -> 6x Motor Port
- P1: DigiKey (none) -> USB4105-GF-A
- R1: value 5.11K -> R5.11K; DigiKey P150BCCT-ND -> RMCF1206FT5K11
- R10, R11, R12, R13, R6, R7, R8, R9: value R150 -> R220; DigiKey P150BCCT-ND -> RMCF1206JT220R
Other:
- moved on the sheet: C10, C12, C14, C2, U3
