File: _autosave-Sheba 2.kicad_pcb (KiCad board)
At the start: 2 copper layers, 85.7 x 54 mm, 63 parts, among them J2 Conn_01x03_Pin, J3 Conn_01x03_Pin, J4 Conn_01x03_Pin, J7 Conn_01x06_Pin, J8 Conn_01x02_Pin, J9 Conn_02x04_Top_Bottom, P1 USB_C_Plug_USB2.0, SW1 SW_SPDT, U1 AP62300TWU, U3 MIC5504-3.3YM5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

Commit message: Getting ready to add overvoltage/ESD protection
Routing:
- net GND: track 41.9 -> 49.8 mm, vias 3 -> 5
