File: _autosave-Sheba 2.kicad_sch (KiCad schematic)
At the start: 66 parts, among them J2 Conn_01x03_Pin, J3 Conn_01x03_Pin, J4 Conn_01x03_Pin, J7 Conn_01x06_Pin, J8 Conn_01x02_Pin, J9 Conn_02x04_Top_Bottom, P1 USB_C_Plug_USB2.0, SW1 SW_SPDT, U1 AP62300TWU, U3 MIC5504-3.3YM5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

Commit message: Getting ready to add overvoltage/ESD protection
Parts:
- removed C11: C2.2uF, Capacitor_SMD:C_1206_3216Metric_Pad1.33x1.80mm_HandSolder, symbol Device:C_Small
- removed C15: C0.1uF, Capacitor_SMD:C_1206_3216Metric_Pad1.33x1.80mm_HandSolder, symbol Device:C_Small
- removed C9: C0.01uF, Capacitor_SMD:C_1206_3216Metric_Pad1.33x1.80mm_HandSolder, symbol Device:C_Small
- removed MT1: ICM-42670-P, Library:XDCR_ICM-42670-P, symbol ICM-42670-P:ICM-42670-P
- removed R4, R5: R10k, Resistor_SMD:R_1206_3216Metric_Pad1.30x1.75mm_HandSolder, symbol Device:R
- D1, D3, D5: value LED Red -> LED Green; DigiKey 150120RS75000 -> 150120VS75000
- D2, D4, D6: value LED Green -> LED Red; DigiKey 150120VS75000 -> 150120RS75000
- J8: footprint Connector_PinHeader_2.54mm:PinHeader_1x02_P2.54mm_Vertical -> Connector_PinHeader_2.54mm:PinHeader_1x03_P2.54mm_Vertical; symbol Connector:Conn_01x02_Pin -> Connector:Conn_01x03_Pin
Connections:
- net GND: now also J8.1 (Pin_1)
- net M1_FWD: now also D1.2 (A); no longer D6.2 (A)
- net M1_REV: now also D2.2 (A); no longer D5.2 (A)
- net M2_FWD: now also D3.2 (A); no longer D4.2 (A)
- net M2_REV: now also D4.2 (A); no longer D3.2 (A)
- net M3_FWD: now also D5.2 (A); no longer D2.2 (A)
- net M3_REV: now also D6.2 (A); no longer D1.2 (A)
- net USART3_TX: now also J8.3 (Pin_3); no longer J8.1 (Pin_1)
- net I2C2_SCL: no longer names the net of U4.26 (PB13)
- net I2C2_SDA: no longer names the net of U4.27 (PB14)
- net IMU_INT: no longer names the net of U4.28 (PB15)
- no-connect marks 12 -> 10
Other:
- note added: "CPU STATUS LED"
- note removed: "AP_CS wired to VDD for I2C mode"
- note removed: "I2C Pull-ups"
- note removed: "IMU - Accel/Gyro/Temp chip ICM-42670-P"
- note removed: "Indicator LEDs"
- moved on the sheet: C10, C12, C14, C16, C17, C18, C2, C3, C4, C5, C6, C7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
